Commit message: modift khr.urdf properties of limits

File: assets/urdf/khr/khr.urdf (robot description, URDF)
Before this commit: robot khr, 18 links, 17 joints
Joints:
- joint HEAD_JOINT0: limit lower=-3.14159 upper=3.14159 effort=0.005 velocity=0.1 -> lower=-1.5708 upper=1.5708 effort=0.005 velocity=1.0
- joint LARM_JOINT0: limit lower=-3.14159 upper=3.14159 effort=0.005 velocity=0.1 -> lower=-1.5708 upper=1.5708 effort=0.005 velocity=1.0
- joint LARM_JOINT1: limit lower=-3.14159 upper=3.14159 effort=0.005 velocity=0.1 -> lower=-1.5708 upper=1.5708 effort=0.005 velocity=1.0
- joint LARM_JOINT2: limit lower=-3.14159 upper=3.14159 effort=0.005 velocity=0.1 -> lower=-1.5708 upper=1.5708 effort=0.005 velocity=1.0
- joint LLEG_JOINT0: limit lower=-3.14159 upper=3.14159 effort=0.005 velocity=0.1 -> lower=-1.5708 upper=1.5708 effort=0.005 velocity=1.0
- joint LLEG_JOINT1: limit lower=-3.14159 upper=3.14159 effort=0.005 velocity=0.1 -> lower=-1.5708 upper=1.5708 effort=0.005 velocity=1.0
- joint LLEG_JOINT2: limit lower=-3.14159 upper=3.14159 effort=0.005 velocity=0.1 -> lower=-1.5708 upper=1.5708 effort=0.005 velocity=1.0
- joint LLEG_JOINT3: limit lower=-3.14159 upper=3.14159 effort=0.005 velocity=0.1 -> lower=-1.5708 upper=1.5708 effort=0.005 velocity=1.0
- joint LLEG_JOINT4: limit lower=-3.14159 upper=3.14159 effort=0.005 velocity=0.1 -> lower=-1.5708 upper=1.5708 effort=0.005 velocity=1.0
- joint RARM_JOINT0: limit lower=-3.14159 upper=3.14159 effort=0.005 velocity=0.1 -> lower=-1.5708 upper=1.5708 effort=0.005 velocity=1.0
- joint RARM_JOINT1: limit lower=-3.14159 upper=3.14159 effort=0.005 velocity=0.1 -> lower=-1.5708 upper=1.5708 effort=0.005 velocity=1.0
- joint RARM_JOINT2: limit lower=-3.14159 upper=3.14159 effort=0.005 velocity=0.1 -> lower=-1.5708 upper=1.5708 effort=0.005 velocity=1.0
- joint RLEG_JOINT0: limit lower=-3.14159 upper=3.14159 effort=0.005 velocity=0.1 -> lower=-1.5708 upper=1.5708 effort=0.005 velocity=1.0
- joint RLEG_JOINT1: limit lower=-3.14159 upper=3.14159 effort=0.005 velocity=0.1 -> lower=-1.5708 upper=1.5708 effort=0.005 velocity=1.0
- joint RLEG_JOINT2: limit lower=-3.14159 upper=3.14159 effort=0.005 velocity=0.1 -> lower=-1.5708 upper=1.5708 effort=0.005 velocity=1.0
- joint RLEG_JOINT3: limit lower=-3.14159 upper=3.14159 effort=0.005 velocity=0.1 -> lower=-1.5708 upper=1.5708 effort=0.005 velocity=1.0
- joint RLEG_JOINT4: limit lower=-3.14159 upper=3.14159 effort=0.005 velocity=0.1 -> lower=-1.5708 upper=1.5708 effort=0.005 velocity=1.0

Commit message: modify config and train scripts

File: assets/urdf/khr/khr.urdf (robot description, URDF)
Before this commit: robot khr, 18 links, 17 joints
Links:
- link BODY: geometry collision mesh filename=khr/mesh/BODY_mesh.obj scale=1 1 1; visual mesh filename=khr/mesh/BODY_mesh.obj scale=1 1 1
- link HEAD_LINK0: geometry collision mesh filename=khr/mesh/HEAD_LINK0_mesh.obj scale=1 1 1; visual mesh filename=khr/mesh/HEAD_LINK0_mesh.obj scale=1 1 1
- link LARM_LINK0: geometry collision mesh filename=khr/mesh/LARM_LINK0_mesh.obj scale=1 1 1; visual mesh filename=khr/mesh/LARM_LINK0_mesh.obj scale=1 1 1
- link LARM_LINK1: geometry collision mesh filename=khr/mesh/LARM_LINK1_mesh.obj scale=1 1 1; visual mesh filename=khr/mesh/LARM_LINK1_mesh.obj scale=1 1 1
- link LARM_LINK2: geometry collision mesh filename=khr/mesh/LARM_LINK2_mesh.obj scale=1 1 1; visual mesh filename=khr/mesh/LARM_LINK2_mesh.obj scale=1 1 1
- link LLEG_LINK0: geometry collision mesh filename=khr/mesh/LLEG_LINK0_mesh.obj scale=1 1 1; visual mesh filename=khr/mesh/LLEG_LINK0_mesh.obj scale=1 1 1
- link LLEG_LINK1: geometry collision mesh filename=khr/mesh/LLEG_LINK1_mesh.obj scale=1 1 1; visual mesh filename=khr/mesh/LLEG_LINK1_mesh.obj scale=1 1 1
- link LLEG_LINK2: geometry collision mesh filename=khr/mesh/LLEG_LINK2_mesh.obj scale=1 1 1; visual mesh filename=khr/mesh/LLEG_LINK2_mesh.obj scale=1 1 1
- link LLEG_LINK3: geometry collision mesh filename=khr/mesh/LLEG_LINK3_mesh.obj scale=1 1 1; visual mesh filename=khr/mesh/LLEG_LINK3_mesh.obj scale=1 1 1
- link LLEG_LINK4: geometry collision mesh filename=khr/mesh/LLEG_LINK4_mesh.obj scale=1 1 1; visual mesh filename=khr/mesh/LLEG_LINK4_mesh.obj scale=1 1 1
- link RARM_LINK0: geometry collision mesh filename=khr/mesh/RARM_LINK0_mesh.obj scale=1 1 1; visual mesh filename=khr/mesh/RARM_LINK0_mesh.obj scale=1 1 1
- link RARM_LINK1: geometry collision mesh filename=khr/mesh/RARM_LINK1_mesh.obj scale=1 1 1; visual mesh filename=khr/mesh/RARM_LINK1_mesh.obj scale=1 1 1
- link RARM_LINK2: geometry collision mesh filename=khr/mesh/RARM_LINK2_mesh.obj scale=1 1 1; visual mesh filename=khr/mesh/RARM_LINK2_mesh.obj scale=1 1 1
- link RLEG_LINK0: geometry collision mesh filename=khr/mesh/RLEG_LINK0_mesh.obj scale=1 1 1; visual mesh filename=khr/mesh/RLEG_LINK0_mesh.obj scale=1 1 1
- link RLEG_LINK1: geometry collision mesh filename=khr/mesh/RLEG_LINK1_mesh.obj scale=1 1 1; visual mesh filename=khr/mesh/RLEG_LINK1_mesh.obj scale=1 1 1
- link RLEG_LINK2: geometry collision mesh filename=khr/mesh/RLEG_LINK2_mesh.obj scale=1 1 1; visual mesh filename=khr/mesh/RLEG_LINK2_mesh.obj scale=1 1 1
- link RLEG_LINK3: geometry collision mesh filename=khr/mesh/RLEG_LINK3_mesh.obj scale=1 1 1; visual mesh filename=khr/mesh/RLEG_LINK3_mesh.obj scale=1 1 1
- link RLEG_LINK4: geometry collision mesh filename=khr/mesh/RLEG_LINK4_mesh.obj scale=1 1 1; visual mesh filename=khr/mesh/RLEG_LINK4_mesh.obj scale=1 1 1

Commit message: create mjcf file for khr retarget and modify urdf

File: assets/urdf/khr/khr.urdf (robot description, URDF)
Before this commit: robot khr, 18 links, 17 joints
Links:
- link BODY: geometry collision mesh filename=mesh/BODY_mesh.stl scale=1 1 1; visual mesh filename=mesh/BODY_mesh.stl scale=1 1 1
- link HEAD_LINK0: geometry collision mesh filename=mesh/HEAD_LINK0_mesh.stl scale=1 1 1; visual mesh filename=mesh/HEAD_LINK0_mesh.stl scale=1 1 1
- link LARM_LINK0: geometry collision mesh filename=mesh/LARM_LINK0_mesh.stl scale=1 1 1; visual mesh filename=mesh/LARM_LINK0_mesh.stl scale=1 1 1
- link LARM_LINK1: geometry collision mesh filename=mesh/LARM_LINK1_mesh.stl scale=1 1 1; visual mesh filename=mesh/LARM_LINK1_mesh.stl scale=1 1 1
- link LARM_LINK2: geometry collision mesh filename=mesh/LARM_LINK2_mesh.stl scale=1 1 1; visual mesh filename=mesh/LARM_LINK2_mesh.stl scale=1 1 1
- link LLEG_LINK0: geometry collision mesh filename=mesh/LLEG_LINK0_mesh.stl scale=1 1 1; visual mesh filename=mesh/LLEG_LINK0_mesh.stl scale=1 1 1
- link LLEG_LINK1: geometry collision mesh filename=mesh/LLEG_LINK1_mesh.stl scale=1 1 1; visual mesh filename=mesh/LLEG_LINK1_mesh.stl scale=1 1 1
- link LLEG_LINK2: geometry collision mesh filename=mesh/LLEG_LINK2_mesh.stl scale=1 1 1; visual mesh filename=mesh/LLEG_LINK2_mesh.stl scale=1 1 1
- link LLEG_LINK3: geometry collision mesh filename=mesh/LLEG_LINK3_mesh.stl scale=1 1 1; visual mesh filename=mesh/LLEG_LINK3_mesh.stl scale=1 1 1
- link LLEG_LINK4: geometry collision mesh filename=mesh/LLEG_LINK4_mesh.stl scale=1 1 1; visual mesh filename=mesh/LLEG_LINK4_mesh.stl scale=1 1 1
- link RARM_LINK0: geometry collision mesh filename=mesh/RARM_LINK0_mesh.stl scale=1 1 1; visual mesh filename=mesh/RARM_LINK0_mesh.stl scale=1 1 1
- link RARM_LINK1: geometry collision mesh filename=mesh/RARM_LINK1_mesh.stl scale=1 1 1; visual mesh filename=mesh/RARM_LINK1_mesh.stl scale=1 1 1
- link RARM_LINK2: geometry collision mesh filename=mesh/RARM_LINK2_mesh.stl scale=1 1 1; visual mesh filename=mesh/RARM_LINK2_mesh.stl scale=1 1 1
- link RLEG_LINK0: geometry collision mesh filename=mesh/RLEG_LINK0_mesh.stl scale=1 1 1; visual mesh filename=mesh/RLEG_LINK0_mesh.stl scale=1 1 1
- link RLEG_LINK1: geometry collision mesh filename=mesh/RLEG_LINK1_mesh.stl scale=1 1 1; visual mesh filename=mesh/RLEG_LINK1_mesh.stl scale=1 1 1
- link RLEG_LINK2: geometry collision mesh filename=mesh/RLEG_LINK2_mesh.stl scale=1 1 1; visual mesh filename=mesh/RLEG_LINK2_mesh.stl scale=1 1 1
- link RLEG_LINK3: geometry collision mesh filename=mesh/RLEG_LINK3_mesh.stl scale=1 1 1; visual mesh filename=mesh/RLEG_LINK3_mesh.stl scale=1 1 1
- link RLEG_LINK4: geometry collision mesh filename=mesh/RLEG_LINK4_mesh.stl scale=1 1 1; visual mesh filename=mesh/RLEG_LINK4_mesh.stl scale=1 1 1

Commit message: update for khr amp

File: assets/urdf/khr/khr.urdf (robot description, URDF)
Before this commit: robot khr, 18 links, 17 joints
Links:
- added link HIP_VIRTUAL_LINK, mass 1e-07
- added link LARM_VIRTUAL_LINK1, mass 1e-07
- added link LARM_VIRTUAL_LINK2, mass 1e-07
- added link LHAND_VIRTUAL_LINK, mass 1e-07
- added link LLEG_VIRTUAL_LINK1, mass 1e-07
- added link LLEG_VIRTUAL_LINK2, mass 1e-07
- added link LLEG_VIRTUAL_LINK3, mass 1e-07
- added link RARM_VIRTUAL_LINK1, mass 1e-07
- added link RARM_VIRTUAL_LINK2, mass 1e-07
- added link RHAND_VIRTUAL_LINK, mass 1e-07
- added link RLEG_VIRTUAL_LINK1, mass 1e-07
- added link RLEG_VIRTUAL_LINK2, mass 1e-07
- added link RLEG_VIRTUAL_LINK3, mass 1e-07
- added link SPINE_VIRTUAL_LINK, mass 1e-07
- added link TORSO_VIRTUAL_LINK, mass 1e-07
- link BODY: geometry collision mesh filename=mesh/BODY_mesh.dae scale=1 1 1; visual mesh filename=mesh/BODY_mesh.dae scale=1 1 1
- link HEAD_LINK0: geometry collision mesh filename=mesh/HEAD_LINK0_mesh.dae scale=1 1 1; visual mesh filename=mesh/HEAD_LINK0_mesh.dae scale=1 1 1
- link LARM_LINK0: geometry collision mesh filename=mesh/LARM_LINK0_mesh.dae scale=1 1 1; visual mesh filename=mesh/LARM_LINK0_mesh.dae scale=1 1 1
- link LARM_LINK1: geometry collision mesh filename=mesh/LARM_LINK1_mesh.dae scale=1 1 1; visual mesh filename=mesh/LARM_LINK1_mesh.dae scale=1 1 1
- link LARM_LINK2: geometry collision mesh filename=mesh/LARM_LINK2_mesh.dae scale=1 1 1; visual mesh filename=mesh/LARM_LINK2_mesh.dae scale=1 1 1
- link LLEG_LINK0: geometry collision mesh filename=mesh/LLEG_LINK0_mesh.dae scale=1 1 1; visual mesh filename=mesh/LLEG_LINK0_mesh.dae scale=1 1 1
- link LLEG_LINK1: geometry collision mesh filename=mesh/LLEG_LINK1_mesh.dae scale=1 1 1; visual mesh filename=mesh/LLEG_LINK1_mesh.dae scale=1 1 1
- link LLEG_LINK2: geometry collision mesh filename=mesh/LLEG_LINK2_mesh.dae scale=1 1 1; visual mesh filename=mesh/LLEG_LINK2_mesh.dae scale=1 1 1
- link LLEG_LINK3: geometry collision mesh filename=mesh/LLEG_LINK3_mesh.dae scale=1 1 1; visual mesh filename=mesh/LLEG_LINK3_mesh.dae scale=1 1 1
- link LLEG_LINK4: geometry collision mesh filename=mesh/LLEG_LINK4_mesh.dae scale=1 1 1; visual mesh filename=mesh/LLEG_LINK4_mesh.dae scale=1 1 1
- link RARM_LINK0: geometry collision mesh filename=mesh/RARM_LINK0_mesh.dae scale=1 1 1; visual mesh filename=mesh/RARM_LINK0_mesh.dae scale=1 1 1
- link RARM_LINK1: geometry collision mesh filename=mesh/RARM_LINK1_mesh.dae scale=1 1 1; visual mesh filename=mesh/RARM_LINK1_mesh.dae scale=1 1 1
- link RARM_LINK2: geometry collision mesh filename=mesh/RARM_LINK2_mesh.dae scale=1 1 1; visual mesh filename=mesh/RARM_LINK2_mesh.dae scale=1 1 1
- link RLEG_LINK0: geometry collision mesh filename=mesh/RLEG_LINK0_mesh.dae scale=1 1 1; visual mesh filename=mesh/RLEG_LINK0_mesh.dae scale=1 1 1
- link RLEG_LINK1: geometry collision mesh filename=mesh/RLEG_LINK1_mesh.dae scale=1 1 1; visual mesh filename=mesh/RLEG_LINK1_mesh.dae scale=1 1 1
- link RLEG_LINK2: geometry collision mesh filename=mesh/RLEG_LINK2_mesh.dae scale=1 1 1; visual mesh filename=mesh/RLEG_LINK2_mesh.dae scale=1 1 1
- link RLEG_LINK3: geometry collision mesh filename=mesh/RLEG_LINK3_mesh.dae scale=1 1 1; visual mesh filename=mesh/RLEG_LINK3_mesh.dae scale=1 1 1
- link RLEG_LINK4: geometry collision mesh filename=mesh/RLEG_LINK4_mesh.dae scale=1 1 1; visual mesh filename=mesh/RLEG_LINK4_mesh.dae scale=1 1 1
Joints:
- added joint HIP_VIRTUAL_JOINT: type fixed, parent HIP_VIRTUAL_LINK, child SPINE_VIRTUAL_LINK, origin xyz=0.0 0.0 0.0 rpy=0.0 0.0 0.0
- added joint LARM_VIRTUAL_JOINT1: type fixed, parent LARM_LINK1, child LARM_VIRTUAL_LINK1, origin xyz=-0.02 0.0 0.0 rpy=0.0 0.0 0.0
- added joint LARM_VIRTUAL_JOINT2: type fixed, parent LARM_LINK2, child LARM_VIRTUAL_LINK2, origin xyz=0.0 0.02 0.0 rpy=0.0 0.0 0.0
- added joint LHAND_VIRTUAL_JOINT: type fixed, parent LARM_LINK2, child LHAND_VIRTUAL_LINK, origin xyz=0.0 0.02 -0.08 rpy=0.0 0.0 0.0
- added joint LLEG_VIRTUAL_JOINT1: type fixed, parent LLEG_LINK1, child LLEG_VIRTUAL_LINK1, origin xyz=0.0 0.02 0.0 rpy=0.0 0.0 0.0
- added joint LLEG_VIRTUAL_JOINT2: type fixed, parent LLEG_LINK2, child LLEG_VIRTUAL_LINK2, origin xyz=0.0 0.02 0.0 rpy=0.0 0.0 0.0
- added joint LLEG_VIRTUAL_JOINT3: type fixed, parent LLEG_LINK3, child LLEG_VIRTUAL_LINK3, origin xyz=0.0 0.02 0.0 rpy=0.0 0.0 0.0
- added joint RARM_VIRTUAL_JOINT1: type fixed, parent RARM_LINK1, child RARM_VIRTUAL_LINK1, origin xyz=-0.02 0.0 0.0 rpy=0.0 0.0 0.0
- added joint RARM_VIRTUAL_JOINT2: type fixed, parent RARM_LINK2, child RARM_VIRTUAL_LINK2, origin xyz=0.0 -0.02 0.0 rpy=0.0 0.0 0.0
- added joint RHAND_VIRTUAL_JOINT: type fixed, parent RARM_LINK2, child RHAND_VIRTUAL_LINK, origin xyz=0.0 -0.02 -0.08 rpy=0.0 0.0 0.0
- added joint RLEG_VIRTUAL_JOINT1: type fixed, parent RLEG_LINK1, child RLEG_VIRTUAL_LINK1, origin xyz=0.0 -0.02 0.0 rpy=0.0 0.0 0.0
- added joint RLEG_VIRTUAL_JOINT2: type fixed, parent RLEG_LINK2, child RLEG_VIRTUAL_LINK2, origin xyz=0.0 -0.02 0.0 rpy=0.0 0.0 0.0
- added joint RLEG_VIRTUAL_JOINT3: type fixed, parent RLEG_LINK3, child RLEG_VIRTUAL_LINK3, origin xyz=0.0 -0.02 0.0 rpy=0.0 0.0 0.0
- added joint SPINE_VIRTUAL_JOINT: type fixed, parent HIP_VIRTUAL_LINK, child BODY, origin xyz=0.0 0.0 0.06265 rpy=0.0 0.0 0.0
- added joint TORSO_VIRTUAL_JOINT: type fixed, parent BODY, child TORSO_VIRTUAL_LINK, origin xyz=0.0 0.0 0.0474 rpy=0.0 0.0 0.0
- joint HEAD_JOINT0: limit lower=-1.5708 upper=1.5708 effort=0.005 velocity=1.0 -> lower=-1.5708 upper=1.5708 effort=2.5 velocity=10.0; origin xyz=0 0 0.0644 rpy=0 -0 0  -> xyz=0 0 0.0170 rpy=0 -0 0 ; parent BODY -> TORSO_VIRTUAL_LINK
- joint LARM_JOINT0: limit lower=-1.5708 upper=1.5708 effort=0.005 velocity=1.0 -> lower=-3.1416 upper=0.5236 effort=2.5 velocity=10.0; origin xyz=0.0115 0.049 0.0474 rpy=0 -0 0  -> xyz=0.0115 0.049 0.0 rpy=0 -0 0 ; parent BODY -> TORSO_VIRTUAL_LINK
- joint LARM_JOINT1: limit lower=-1.5708 upper=1.5708 effort=0.005 velocity=1.0 -> lower=-0.5236 upper=3.1416 effort=2.5 velocity=10.0
- joint LARM_JOINT2: limit lower=-1.5708 upper=1.5708 effort=0.005 velocity=1.0 -> lower=-2.0944 upper=0.0 effort=2.5 velocity=10.0
- joint LLEG_JOINT0: limit lower=-1.5708 upper=1.5708 effort=0.005 velocity=1.0 -> lower=-0.2618 upper=0.5236 effort=2.5 velocity=10.0; origin xyz=0.018517 0.017 -0.06265 rpy=0 -0 0  -> xyz=0.018517 0.017 0.0 rpy=0 -0 0 ; parent BODY -> HIP_VIRTUAL_LINK
- joint LLEG_JOINT1: limit lower=-1.5708 upper=1.5708 effort=0.005 velocity=1.0 -> lower=-1.5708 upper=1.5708 effort=2.5 velocity=10.0
- joint LLEG_JOINT2: limit lower=-1.5708 upper=1.5708 effort=0.005 velocity=1.0 -> lower=0.0 upper=2.6180 effort=2.5 velocity=10.0
- joint LLEG_JOINT3: limit lower=-1.5708 upper=1.5708 effort=0.005 velocity=1.0 -> lower=0.0 upper=1.5708 effort=2.5 velocity=10.0
- joint LLEG_JOINT4: limit lower=-1.5708 upper=1.5708 effort=0.005 velocity=1.0 -> lower=-0.5236 upper=0.0 effort=2.5 velocity=10.0
- joint RARM_JOINT0: limit lower=-1.5708 upper=1.5708 effort=0.005 velocity=1.0 -> lower=-3.1416 upper=0.5236 effort=2.5 velocity=10.0; origin xyz=0.0115 -0.049 0.0474 rpy=0 -0 0  -> xyz=0.0115 -0.049 0.0 rpy=0 -0 0 ; parent BODY -> TORSO_VIRTUAL_LINK
- joint RARM_JOINT1: limit lower=-1.5708 upper=1.5708 effort=0.005 velocity=1.0 -> lower=-3.1416 upper=0.5236 effort=2.5 velocity=10.0
- joint RARM_JOINT2: limit lower=-1.5708 upper=1.5708 effort=0.005 velocity=1.0 -> lower=-2.0944 upper=0.0 effort=2.5 velocity=10.0
- joint RLEG_JOINT0: limit lower=-1.5708 upper=1.5708 effort=0.005 velocity=1.0 -> lower=-0.5236 upper=0.2518 effort=2.5 velocity=10.0; origin xyz=0.018517 -0.017 -0.06265 rpy=0 -0 0  -> xyz=0.018517 -0.017 0.0 rpy=0 -0 0 ; parent BODY -> HIP_VIRTUAL_LINK
- joint RLEG_JOINT1: limit lower=-1.5708 upper=1.5708 effort=0.005 velocity=1.0 -> lower=-1.5708 upper=1.5708 effort=2.5 velocity=10.0
- joint RLEG_JOINT2: limit lower=-1.5708 upper=1.5708 effort=0.005 velocity=1.0 -> lower=0.0 upper=2.6108 effort=2.5 velocity=10.0
- joint RLEG_JOINT3: limit lower=-1.5708 upper=1.5708 effort=0.005 velocity=1.0 -> lower=0.0 upper=1.5708 effort=2.5 velocity=10.0
- joint RLEG_JOINT4: limit lower=-1.5708 upper=1.5708 effort=0.005 velocity=1.0 -> lower=0.0 upper=0.5236 effort=2.5 velocity=10.0
