Commit message: debug

File: assets/urdf/khr/khr_set_limit_joint.urdf (robot description, URDF)
Before this commit: robot khr, 18 links, 17 joints
Joints:
- joint LARM_JOINT0: limit lower=-3.1416 upper=0.5236 effort=2.5 velocity=10.0 -> lower=-3.1416 upper=0.7854 effort=2.5 velocity=10.0
- joint LLEG_JOINT3: limit lower=0.0 upper=1.5708 effort=2.5 velocity=10.0 -> lower=-1.8326 upper=2.3561 effort=2.5 velocity=10.0
- joint RARM_JOINT0: limit lower=-3.1416 upper=0.5236 effort=2.5 velocity=10.0 -> lower=-3.1416 upper=0.7854 effort=2.5 velocity=10.0
- joint RLEG_JOINT0: limit lower=-0.5236 upper=0.2518 effort=2.5 velocity=10.0 -> lower=-0.5236 upper=0.2618 effort=2.5 velocity=10.0
- joint RLEG_JOINT3: limit lower=0.0 upper=1.5708 effort=2.5 velocity=10.0 -> lower=-1.8326 upper=2.3561 effort=2.5 velocity=10.0
