Commit message: add khr model with small foot

File: assets/urdf/khr/khr_set_limit_joint_w_small_foot.urdf (robot description, URDF)
Before this commit: robot khr, 18 links, 17 joints
Links:
- link LLEG_LINK4: geometry collision mesh filename=khr/mesh/LLEG_LINK4_mesh_sole.dae scale=1 1 1; visual mesh filename=khr/mesh/LLEG_LINK4_mesh_sole.dae scale=1 1 1
- link RLEG_LINK4: geometry collision mesh filename=khr/mesh/RLEG_LINK4_mesh_sole.dae scale=1 1 1; visual mesh filename=khr/mesh/RLEG_LINK4_mesh_sole.dae scale=1 1 1

File: assets/urdf/khr/khr_set_limit_joint_w_small_foot_ver1.urdf (robot description, URDF)
Before this commit: robot khr, 18 links, 17 joints
Links:
- link LLEG_LINK4: geometry collision mesh filename=khr/mesh/LLEG_LINK4_mesh_sole_ver1.dae scale=1 1 1; visual mesh filename=khr/mesh/LLEG_LINK4_mesh_sole_ver1.dae scale=1 1 1
- link RLEG_LINK4: geometry collision mesh filename=khr/mesh/RLEG_LINK4_mesh_sole_ver1.dae scale=1 1 1; visual mesh filename=khr/mesh/RLEG_LINK4_mesh_sole_ver1.dae scale=1 1 1
