Commit message: update

File: assets/urdf/khr/khr22/khr22_refined_mesh_original_foot.urdf (robot description, URDF)
Before this commit: robot khr22, 23 links, 22 joints
Links:
- link LLEG_LINK5: geometry collision mesh filename=khr22/mesh/LLEG_LINK5_mesh.dae scale=1 1 1; visual mesh filename=khr22/mesh/LLEG_LINK5_mesh.dae scale=1 1 1
- link RLEG_LINK5: geometry collision mesh filename=khr22/mesh/RLEG_LINK5_mesh.dae scale=1 1 1; visual mesh filename=khr22/mesh/RLEG_LINK5_mesh.dae scale=1 1 1

File: isaacgymenvs/motion_retarget/assets/urdf/khr/khr_set_limit_joint.urdf (robot description, URDF)
Before this commit: robot khr, 33 links, 32 joints
Links:
- removed link HIP_VIRTUAL_LINK
- removed link LARM_VIRTUAL_LINK1
- removed link LARM_VIRTUAL_LINK2
- removed link LHAND_VIRTUAL_LINK
- removed link LLEG_VIRTUAL_LINK1
- removed link LLEG_VIRTUAL_LINK2
- removed link LLEG_VIRTUAL_LINK3
- removed link RARM_VIRTUAL_LINK1
- removed link RARM_VIRTUAL_LINK2
- removed link RHAND_VIRTUAL_LINK
- removed link RLEG_VIRTUAL_LINK1
- removed link RLEG_VIRTUAL_LINK2
- removed link RLEG_VIRTUAL_LINK3
- removed link SPINE_VIRTUAL_LINK
- removed link TORSO_VIRTUAL_LINK
- link BODY: geometry collision mesh filename=khr/mesh/BODY_mesh.dae scale=1 1 1; visual mesh filename=khr/mesh/BODY_mesh.dae scale=1 1 1
- link HEAD_LINK0: geometry collision mesh filename=khr/mesh/HEAD_LINK0_mesh.dae scale=1 1 1; visual mesh filename=khr/mesh/HEAD_LINK0_mesh.dae scale=1 1 1
- link LARM_LINK0: geometry collision mesh filename=khr/mesh/LARM_LINK0_mesh.dae scale=1 1 1; visual mesh filename=khr/mesh/LARM_LINK0_mesh.dae scale=1 1 1
- link LARM_LINK1: geometry collision mesh filename=khr/mesh/LARM_LINK1_mesh.dae scale=1 1 1; visual mesh filename=khr/mesh/LARM_LINK1_mesh.dae scale=1 1 1
- link LARM_LINK2: geometry collision mesh filename=khr/mesh/LARM_LINK2_mesh.dae scale=1 1 1; visual mesh filename=khr/mesh/LARM_LINK2_mesh.dae scale=1 1 1
- link LLEG_LINK0: geometry collision mesh filename=khr/mesh/LLEG_LINK0_mesh.dae scale=1 1 1; visual mesh filename=khr/mesh/LLEG_LINK0_mesh.dae scale=1 1 1
- link LLEG_LINK1: geometry collision mesh filename=khr/mesh/LLEG_LINK1_mesh.dae scale=1 1 1; visual mesh filename=khr/mesh/LLEG_LINK1_mesh.dae scale=1 1 1
- link LLEG_LINK2: geometry collision mesh filename=khr/mesh/LLEG_LINK2_mesh.dae scale=1 1 1; visual mesh filename=khr/mesh/LLEG_LINK2_mesh.dae scale=1 1 1
- link LLEG_LINK3: geometry collision mesh filename=khr/mesh/LLEG_LINK3_mesh.dae scale=1 1 1; visual mesh filename=khr/mesh/LLEG_LINK3_mesh.dae scale=1 1 1
- link LLEG_LINK4: geometry collision mesh filename=khr/mesh/LLEG_LINK4_mesh.dae scale=1 1 1; visual mesh filename=khr/mesh/LLEG_LINK4_mesh.dae scale=1 1 1
- link RARM_LINK0: geometry collision mesh filename=khr/mesh/RARM_LINK0_mesh.dae scale=1 1 1; visual mesh filename=khr/mesh/RARM_LINK0_mesh.dae scale=1 1 1
- link RARM_LINK1: geometry collision mesh filename=khr/mesh/RARM_LINK1_mesh.dae scale=1 1 1; visual mesh filename=khr/mesh/RARM_LINK1_mesh.dae scale=1 1 1
- link RARM_LINK2: geometry collision mesh filename=khr/mesh/RARM_LINK2_mesh.dae scale=1 1 1; visual mesh filename=khr/mesh/RARM_LINK2_mesh.dae scale=1 1 1
- link RLEG_LINK0: geometry collision mesh filename=khr/mesh/RLEG_LINK0_mesh.dae scale=1 1 1; visual mesh filename=khr/mesh/RLEG_LINK0_mesh.dae scale=1 1 1
- link RLEG_LINK1: geometry collision mesh filename=khr/mesh/RLEG_LINK1_mesh.dae scale=1 1 1; visual mesh filename=khr/mesh/RLEG_LINK1_mesh.dae scale=1 1 1
- link RLEG_LINK2: geometry collision mesh filename=khr/mesh/RLEG_LINK2_mesh.dae scale=1 1 1; visual mesh filename=khr/mesh/RLEG_LINK2_mesh.dae scale=1 1 1
- link RLEG_LINK3: geometry collision mesh filename=khr/mesh/RLEG_LINK3_mesh.dae scale=1 1 1; visual mesh filename=khr/mesh/RLEG_LINK3_mesh.dae scale=1 1 1
- link RLEG_LINK4: geometry collision mesh filename=khr/mesh/RLEG_LINK4_mesh.dae scale=1 1 1; visual mesh filename=khr/mesh/RLEG_LINK4_mesh.dae scale=1 1 1
Joints:
- removed joint HIP_VIRTUAL_JOINT
- removed joint LARM_VIRTUAL_JOINT1
- removed joint LARM_VIRTUAL_JOINT2
- removed joint LHAND_VIRTUAL_JOINT
- removed joint LLEG_VIRTUAL_JOINT1
- removed joint LLEG_VIRTUAL_JOINT2
- removed joint LLEG_VIRTUAL_JOINT3
- removed joint RARM_VIRTUAL_JOINT1
- removed joint RARM_VIRTUAL_JOINT2
- removed joint RHAND_VIRTUAL_JOINT
- removed joint RLEG_VIRTUAL_JOINT1
- removed joint RLEG_VIRTUAL_JOINT2
- removed joint RLEG_VIRTUAL_JOINT3
- removed joint SPINE_VIRTUAL_JOINT
- removed joint TORSO_VIRTUAL_JOINT
- joint HEAD_JOINT0: limit lower=-1.5708 upper=1.5708 effort=2.5 velocity=10.0 -> lower=-1.5708 upper=1.5708 effort=0.005 velocity=1.0; origin xyz=0 0 0.0170 rpy=0 -0 0  -> xyz=0 0 0.0644 rpy=0 -0 0 ; parent TORSO_VIRTUAL_LINK -> BODY
- joint LARM_JOINT0: limit lower=-3.1416 upper=0.5236 effort=2.5 velocity=10.0 -> lower=-3.1416 upper=0.7854 effort=2.5 velocity=10.0; origin xyz=0.0115 0.049 0.0 rpy=0 -0 0  -> xyz=0.0115 0.049 0.0474 rpy=0 -0 0 ; parent TORSO_VIRTUAL_LINK -> BODY
- joint LLEG_JOINT0: origin xyz=0.018517 0.017 0.0 rpy=0 -0 0  -> xyz=0.018517 0.017 -0.06265 rpy=0 -0 0 ; parent HIP_VIRTUAL_LINK -> BODY
- joint LLEG_JOINT3: limit lower=0.0 upper=1.5708 effort=2.5 velocity=10.0 -> lower=-1.8326 upper=2.3561 effort=2.5 velocity=10.0
- joint RARM_JOINT0: limit lower=-3.1416 upper=0.5236 effort=2.5 velocity=10.0 -> lower=-3.1416 upper=0.7854 effort=2.5 velocity=10.0; origin xyz=0.0115 -0.049 0.0 rpy=0 -0 0  -> xyz=0.0115 -0.049 0.0474 rpy=0 -0 0 ; parent TORSO_VIRTUAL_LINK -> BODY
- joint RLEG_JOINT0: limit lower=-0.5236 upper=0.2518 effort=2.5 velocity=10.0 -> lower=-0.5236 upper=0.2618 effort=2.5 velocity=10.0; origin xyz=0.018517 -0.017 0.0 rpy=0 -0 0  -> xyz=0.018517 -0.017 -0.06265 rpy=0 -0 0 ; parent HIP_VIRTUAL_LINK -> BODY
- joint RLEG_JOINT3: limit lower=0.0 upper=1.5708 effort=2.5 velocity=10.0 -> lower=-1.8326 upper=2.3561 effort=2.5 velocity=10.0

File: isaacgymenvs/motion_retarget/assets/urdf/khr/khr_set_limit_joint_w_virtual.urdf (robot description, URDF)
Before this commit: robot khr, 33 links, 32 joints
Joints:
- joint HEAD_JOINT0: limit lower=-1.5708 upper=1.5708 effort=1.0 velocity=10.0 -> lower=-1.5708 upper=1.5708 effort=2.5 velocity=10.0
- joint HIP_VIRTUAL_JOINT: origin xyz=0.0 0.0 0.0 rpy=0.0 0.0 0.0 -> xyz=0.0 0.0 0.03 rpy=0.0 0.0 0.0
- joint LARM_JOINT0: limit lower=-3.1416 upper=0.5236 effort=1.0 velocity=10.0 -> lower=-3.1416 upper=0.7854 effort=2.5 velocity=10.0
- joint LARM_JOINT1: limit lower=-0.5236 upper=3.1416 effort=1.0 velocity=10.0 -> lower=-0.5236 upper=3.1416 effort=2.5 velocity=10.0
- joint LARM_JOINT2: limit lower=-2.0944 upper=0.0 effort=1.0 velocity=10.0 -> lower=-2.0944 upper=0.0 effort=2.5 velocity=10.0
- joint LLEG_JOINT0: limit lower=-0.2618 upper=0.5236 effort=1.0 velocity=10.0 -> lower=-0.2618 upper=0.5236 effort=2.5 velocity=10.0
- joint LLEG_JOINT1: limit lower=-1.5708 upper=1.5708 effort=1.0 velocity=10.0 -> lower=-1.5708 upper=1.5708 effort=2.5 velocity=10.0
- joint LLEG_JOINT2: limit lower=0.0 upper=2.6180 effort=1.0 velocity=10.0 -> lower=0.0 upper=2.6180 effort=2.5 velocity=10.0
- joint LLEG_JOINT3: limit lower=0.0 upper=1.5708 effort=1.0 velocity=10.0 -> lower=-1.8326 upper=2.3561 effort=2.5 velocity=10.0
- joint LLEG_JOINT4: limit lower=-0.5236 upper=0.0 effort=1.0 velocity=10.0 -> lower=-0.5236 upper=0.0 effort=2.5 velocity=10.0
- joint RARM_JOINT0: limit lower=-3.1416 upper=0.5236 effort=1.0 velocity=10.0 -> lower=-3.1416 upper=0.7854 effort=2.5 velocity=10.0
- joint RARM_JOINT1: limit lower=-3.1416 upper=0.5236 effort=1.0 velocity=10.0 -> lower=-3.1416 upper=0.5236 effort=2.5 velocity=10.0
- joint RARM_JOINT2: limit lower=-2.0944 upper=0.0 effort=1.0 velocity=10.0 -> lower=-2.0944 upper=0.0 effort=2.5 velocity=10.0
- joint RLEG_JOINT0: limit lower=-0.5236 upper=0.2518 effort=1.0 velocity=10.0 -> lower=-0.5236 upper=0.2618 effort=2.5 velocity=10.0
- joint RLEG_JOINT1: limit lower=-1.5708 upper=1.5708 effort=1.0 velocity=10.0 -> lower=-1.5708 upper=1.5708 effort=2.5 velocity=10.0
- joint RLEG_JOINT2: limit lower=0.0 upper=2.6108 effort=1.0 velocity=10.0 -> lower=0.0 upper=2.6108 effort=2.5 velocity=10.0
- joint RLEG_JOINT3: limit lower=0.0 upper=1.5708 effort=1.0 velocity=10.0 -> lower=-1.8326 upper=2.3561 effort=2.5 velocity=10.0
- joint RLEG_JOINT4: limit lower=0.0 upper=0.5236 effort=1.0 velocity=10.0 -> lower=0.0 upper=0.5236 effort=2.5 velocity=10.0
- joint SPINE_VIRTUAL_JOINT: origin xyz=0.0 0.0 0.06265 rpy=0.0 0.0 0.0 -> xyz=0.0 0.0 0.03265 rpy=0.0 0.0 0.0; parent HIP_VIRTUAL_LINK -> SPINE_VIRTUAL_LINK
