Commit message: add kinova env

File: assets/urdf/kinova/gen3_robotiq_2f_140_backup.urdf (robot description, URDF)
Before this commit: robot gen3_robotiq_2f_140, 24 links, 23 joints
Joints:
- joint joint_1: limit lower=-3.141592 upper=3.14152 effort=39 velocity=1.3963 -> effort=39 velocity=1.3963; type revolute -> continuous
- joint joint_3: limit lower=-3.141592 upper=3.141592 effort=39 velocity=1.3963 -> effort=39 velocity=1.3963; type revolute -> continuous
- joint joint_5: limit lower=-3.141592 upper=3.141592 effort=9 velocity=1.2218 -> effort=9 velocity=1.2218; type revolute -> continuous
- joint joint_7: limit lower=-3.141592 upper=3.141592 effort=9 velocity=1.2218 -> effort=9 velocity=1.2218; type revolute -> continuous
- joint left_inner_finger_joint: limit lower=0 upper=0.8757 effort=1000 velocity=2.0 -> lower=-0.8757 upper=0.8757 effort=1000 velocity=2.0
- joint left_inner_knuckle_joint: limit lower=-0.8757 upper=0 effort=1000 velocity=2.0 -> lower=-0.8757 upper=0.8757 effort=1000 velocity=2.0
- joint right_inner_finger_joint: limit lower=0 upper=0.8757 effort=1000 velocity=2.0 -> lower=-0.8757 upper=0.8757 effort=1000 velocity=2.0
- joint right_inner_knuckle_joint: limit lower=-0.8757 upper=0 effort=1000 velocity=2.0 -> lower=-0.8757 upper=0.8757 effort=1000 velocity=2.0
- joint right_outer_knuckle_joint: limit lower=-0.725 upper=0 effort=1000 velocity=2.0 -> lower=-0.725 upper=0.725 effort=1000 velocity=2.0
