Commit message: fix path of meshes

File: assets/urdf/a0b/A0B.urdf (robot description, URDF)
Before this commit: robot A0B, 7 links, 6 joints
Links:
- link BODY: geometry collision mesh filename=A0B_meshes/BODY_mesh.dae scale=1 1 1; visual mesh filename=A0B_meshes/BODY_mesh.dae scale=1 1 1
- link RARM_LINK0: geometry collision mesh filename=A0B_meshes/RARM_LINK0_mesh.dae scale=1 1 1; visual mesh filename=A0B_meshes/RARM_LINK0_mesh.dae scale=1 1 1
- link RARM_LINK1: geometry collision mesh filename=A0B_meshes/RARM_LINK1_mesh.dae scale=1 1 1; visual mesh filename=A0B_meshes/RARM_LINK1_mesh.dae scale=1 1 1
- link RARM_LINK2: geometry collision mesh filename=A0B_meshes/RARM_LINK2_mesh.dae scale=1 1 1; visual mesh filename=A0B_meshes/RARM_LINK2_mesh.dae scale=1 1 1
- link RARM_LINK3: geometry collision mesh filename=A0B_meshes/RARM_LINK3_mesh.dae scale=1 1 1; visual mesh filename=A0B_meshes/RARM_LINK3_mesh.dae scale=1 1 1
- link RARM_LINK4: geometry collision mesh filename=A0B_meshes/RARM_LINK4_mesh.dae scale=1 1 1; visual mesh filename=A0B_meshes/RARM_LINK4_mesh.dae scale=1 1 1
- link RARM_LINK5: geometry collision mesh filename=A0B_meshes/RARM_LINK5_mesh.dae scale=1 1 1; visual mesh filename=A0B_meshes/RARM_LINK5_mesh.dae scale=1 1 1
